Commit message: uav flies dron

File: grvc-ual/arm_description/models/aeroarms_hecatonquiros_positioner_gripper/arm.transmission.xacro (robot description, xacro)
@@ -116,3 +116,54 @@
     </actuator>
 </transmission>
+<!--Supuestamente las articulaciones de abajo son libres, desactivalas cuando quieras-->
+<transmission name="tran_right/Positioner_HAND_joint">
+    <type>transmission_interface/SimpleTransmission</type>
+    <joint name="right/Positioner_HAND_joint">
+      <hardwareInterface>hardware_interface/EffortJointInterface</hardwareInterface>
+    </joint>
+    <actuator name="motor_right/Positioner_HAND_joint">
+      <hardwareInterface>hardware_interface/EffortJointInterface</hardwareInterface>
+      <mechanicalReduction>1</mechanicalReduction>
+    </actuator>
+</transmission>
+<transmission name="tran_right/Positioner_1_joint">
+    <type>transmission_interface/SimpleTransmission</type>
+    <joint name="right/Positioner_1_joint">
+      <hardwareInterface>hardware_interface/EffortJointInterface</hardwareInterface>
+    </joint>
+    <actuator name="motor_right/Positioner_1_joint">
+      <hardwareInterface>hardware_interface/EffortJointInterface</hardwareInterface>
+      <mechanicalReduction>1</mechanicalReduction>
+    </actuator>
+</transmission>
+<transmission name="tran_right/Positioner_2_joint">
+    <type>transmission_interface/SimpleTransmission</type>
+    <joint name="right/Positioner_2_joint">
+      <hardwareInterface>hardware_interface/EffortJointInterface</hardwareInterface>
+    </joint>
+    <actuator name="motor_right/Positioner_2_joint">
+      <hardwareInterface>hardware_interface/EffortJointInterface</hardwareInterface>
+      <mechanicalReduction>1</mechanicalReduction>
+    </actuator>
+</transmission>
+<transmission name="tran_right/Positioner_BASE_joint">
+    <type>transmission_interface/SimpleTransmission</type>
+    <joint name="right/Positioner_BASE_joint">
+      <hardwareInterface>hardware_interface/EffortJointInterface</hardwareInterface>
+    </joint>
+    <actuator name="motor_right/Positioner_BASE_joint">
+      <hardwareInterface>hardware_interface/EffortJointInterface</hardwareInterface>
+      <mechanicalReduction>1</mechanicalReduction>
+    </actuator>
+</transmission>
+<transmission name="tran_right/Positioner_Fija_BASE_joint">
+    <type>transmission_interface/SimpleTransmission</type>
+    <joint name="right/Positioner_Fija_BASE_joint">
+      <hardwareInterface>hardware_interface/EffortJointInterface</hardwareInterface>
+    </joint>
+    <actuator name="motor_right/Positioner_Fija_BASE_joint">
+      <hardwareInterface>hardware_interface/EffortJointInterface</hardwareInterface>
+      <mechanicalReduction>1</mechanicalReduction>
+    </actuator>
+</transmission>
 </robot>

File: grvc-ual/arm_description/urdf/positioner_gripper.xacro (robot description, xacro)
@@ -1205,3 +1205,53 @@
     </actuator>
   </transmission>
+<!--transmission name="tran_right/Positioner_HAND_joint">
+    <type>transmission_interface/SimpleTransmission</type>
+    <joint name="right/Positioner_HAND_joint">
+      <hardwareInterface>hardware_interface/EffortJointInterface</hardwareInterface>
+    </joint>
+    <actuator name="motor_right/Positioner_HAND_joint">
+      <hardwareInterface>hardware_interface/EffortJointInterface</hardwareInterface>
+      <mechanicalReduction>1</mechanicalReduction>
+    </actuator>
+</transmission>
+<transmission name="tran_right/Positioner_1_joint">
+    <type>transmission_interface/SimpleTransmission</type>
+    <joint name="right/Positioner_1_joint">
+      <hardwareInterface>hardware_interface/EffortJointInterface</hardwareInterface>
+    </joint>
+    <actuator name="motor_right/Positioner_1_joint">
+      <hardwareInterface>hardware_interface/EffortJointInterface</hardwareInterface>
+      <mechanicalReduction>1</mechanicalReduction>
+    </actuator>
+</transmission>
+<transmission name="tran_right/Positioner_2_joint">
+    <type>transmission_interface/SimpleTransmission</type>
+    <joint name="right/Positioner_2_joint">
+      <hardwareInterface>hardware_interface/EffortJointInterface</hardwareInterface>
+    </joint>
+    <actuator name="motor_right/Positioner_2_joint">
+      <hardwareInterface>hardware_interface/EffortJointInterface</hardwareInterface>
+      <mechanicalReduction>1</mechanicalReduction>
+    </actuator>
+</transmission>
+<transmission name="tran_right/Positioner_BASE_joint">
+    <type>transmission_interface/SimpleTransmission</type>
+    <joint name="right/Positioner_BASE_joint">
+      <hardwareInterface>hardware_interface/EffortJointInterface</hardwareInterface>
+    </joint>
+    <actuator name="motor_right/Positioner_BASE_joint">
+      <hardwareInterface>hardware_interface/EffortJointInterface</hardwareInterface>
+      <mechanicalReduction>1</mechanicalReduction>
+    </actuator>
+</transmission-->
+<transmission name="tran_right/Positioner_Fija_BASE_joint">
+    <type>transmission_interface/SimpleTransmission</type>
+    <joint name="right/Positioner_Fija_BASE_joint">
+      <hardwareInterface>hardware_interface/EffortJointInterface</hardwareInterface>
+    </joint>
+    <actuator name="motor_right/Positioner_Fija_BASE_joint">
+      <hardwareInterface>hardware_interface/EffortJointInterface</hardwareInterface>
+      <mechanicalReduction>1</mechanicalReduction>
+    </actuator>
+</transmission>
 </robot>
