Commit message: docker works better

File: grvc-ual/arm_description/urdf/multirotor_base.xacro (robot description, xacro)
@@ -50,15 +50,13 @@
       </collision>
     </link>
-<link name="base_link_inertia_collision_one">
-      <inertial>
-        <mass value="0.01" />  <!-- [kg] QUE HACEMOS AHORA CON LAS MASAS?????????????????????-->
-        <origin xyz="0 0 0" />
-        <xacro:insert_block name="inertia" />
-      </inertial>
-      <collision>
-        <origin xyz="0 0.4 -0.7" rpy="0 0 1.57" />   <!--izquierda-->
-	<!--origin xyz="0 0.2 -0.283" rpy="0 0 0" /-->
-        <geometry>
-	<!--box size="0.28 0.02 0.02" /-->
+<!--link name="base_link_inertia_collision_one">
+      <inertial>
+        <mass value="0.01" />
+        <origin xyz="0 0 0" />
+        <xacro:insert_block name="inertia" />
+      </inertial>
+      <collision>
+        <origin xyz="0 0.4 -0.7" rpy="0 0 1.57" />
+        <geometry>
 	<box size="0.04 1.25 1" />
         </geometry>
@@ -72,13 +70,11 @@
 <link name="base_link_inertia_collision_two">
       <inertial>
-        <mass value="0.01" />  <!-- [kg] QUE HACEMOS AHORA CON LAS MASAS?????????????????????-->
-        <origin xyz="0 0 0" />
-        <xacro:insert_block name="inertia" />
-      </inertial>
-      <collision>
-	<!--origin xyz="0 -0.2 -0.283" rpy="0 0 0" /-->
+        <mass value="0.01" />
+        <origin xyz="0 0 0" />
+        <xacro:insert_block name="inertia" />
+      </inertial>
+      <collision>
         <origin xyz="0 -0.4 -0.7" rpy="0 0 1.57" />
         <geometry>
-	<!--box size="0.28 0.02 0.02" /-->
 	<box size="0.04 1.25 1" />
         </geometry>
@@ -89,5 +85,5 @@
       <parent link="base_link" />
       <child link="base_link_inertia_collision_two" />
-    </joint>
+    </joint-->
 <link name="base_link_inertia_collision_three">
       <inertial>

File: grvc-ual/arm_description/urdf/positioner_gripper.xacro (robot description, xacro)
@@ -1205,5 +1205,5 @@
     </actuator>
   </transmission>
-<!--transmission name="tran_right/Positioner_HAND_joint">
+<transmission name="tran_right/Positioner_HAND_joint">
     <type>transmission_interface/SimpleTransmission</type>
     <joint name="right/Positioner_HAND_joint">
@@ -1244,5 +1244,5 @@
       <mechanicalReduction>1</mechanicalReduction>
     </actuator>
-</transmission-->
+</transmission>
 <transmission name="tran_right/Positioner_Fija_BASE_joint">
     <type>transmission_interface/SimpleTransmission</type>
